Commit message: update lidar position in urdf

File: wamv_nctu_description/urdf/wamv_nctu_description.urdf (robot description, URDF)
Before this commit: robot wamv_nctu_description, 4 links, 3 joints
Joints:
- joint velodyne_joint: origin xyz=0.726949065473584 -0.00179242971869779 1.7318731085397 rpy=0.00101786889643677 0.00151157105591378 0 -> xyz=0.9 -0.00179242971869779 1.3 rpy=0.00101786889643677 0.00151157105591378 0
