Commit message: update motor code

File: wamv_nycu_description/urdf/wamv_nycu_description.urdf (robot description, URDF)
Before this commit: robot wamv_nycu_description, 5 links, 4 joints
Joints:
- joint zed_mid_joint: origin xyz=0.97872 0.058938 1.5612 rpy=0 0.20769 0 -> xyz=0.97872 0.058938 1.5612 rpy=0 0 0
